Commit message: - Adjusted 'update_rate' for IMU

File: sensors_mine_explorer/sensors_mine_explorer_description/urdf/imu/imu.xacro (robot description, xacro)
@@ -12,5 +12,6 @@
           <box size="0.01 0.01 0.005"/>
         </geometry>
-        <material name="orange"><color rgba="1 0.5 0 1"/></material>
+        <material name="orange">
+        <color rgba="1 0.5 0 1"/></material>
       </visual>
     </link>
@@ -18,5 +19,5 @@
       <sensor name="${name}" type="imu">
         <always_on>true</always_on>
-        <update_rate>100</update_rate>
+        <update_rate>30.0</update_rate>
         <visualize>true</visualize>
         <imu>
